File: n9-uart-adapter.kicad_pcb (KiCad board)
At the start: 2 copper layers, 14.4 x 33 mm, 7 parts, among them P1 PAD, P2 PAD, P3 PAD, P4 PAD, P5 PAD, P6 SPRING_FINGERS_1, P7 SPRING_FINGERS_2

Commit message: update
Parts:
- added C1: 100nF, Capacitors_SMD:C_0805, F.Cu at (42.0, 76.6)
- added C2: 10uF, Capacitors_SMD:C_0805, F.Cu at (43.0, 69.4)
- added P8: CONN_01X04, Pin_Headers:Pin_Header_Angled_1x04, F.Cu at (62.9, 75.6)
- added Q1: BSS138, TO_SOT_Packages_SMD:SOT-23, F.Cu at (45.1, 72.3)
- added Q2: BSS138, TO_SOT_Packages_SMD:SOT-23, F.Cu at (51.9, 70.7)
- added R1: 10k, Resistors_SMD:R_0805, F.Cu at (42.0, 72.3)
- added R2: 10k, Resistors_SMD:R_0805, F.Cu at (48.9, 70.7)
- added R3: 10k, Resistors_SMD:R_0805, F.Cu at (61.8, 72.7)
- added R4: 10k, Resistors_SMD:R_0805, F.Cu at (57.8, 72.0)
- added U1: LD1117S18CTR, TO_SOT_Packages_SMD:SOT-223, F.Cu at (35.4, 75.0)
- moved P2 28.3 mm to (47.7, 45.2)
- moved P3 28.3 mm to (50.2, 45.2)
- moved P1 28.3 mm to (45.0, 45.2)
- moved P4 28.3 mm to (50.2, 53.0)
- moved P5 28.3 mm to (45.0, 53.0)
- moved P6 28.3 mm to (47.9, 58.8)
- moved P7 28.3 mm to (47.9, 63.8)
Connections:
- P6 pad 7: (no net) -> GND
- P6 pad 8: (no net) -> /UART3_RX
- P7 pad 7: (no net) -> GND
- P7 pad 8: (no net) -> /UART3_TX
Routing:
- net +5V: track 0.00 -> 48.2 mm
- net GND: track 0.00 -> 43.7 mm, vias 0 -> 2
- net /UART3_RX: track 0.00 -> 27.0 mm, vias 0 -> 2
- net /PC_UART_TX: track 0.00 -> 23.7 mm, vias 0 -> 2
- net +1V8: track 0.00 -> 20.9 mm
- net /UART3_TX: track 0.00 -> 14.5 mm, vias 0 -> 2
- net /PC_UART_RX: track 0.00 -> 8.84 mm
Other:
- board size 14.4 x 33 mm -> 35 x 40 mm
