File: n9-uart-adapter.sch (KiCad schematic (older format))
At the start: 7 parts, among them P1 PAD, P2 PAD, P3 PAD, P4 PAD, P5 PAD, P6 SPRING_FINGERS_1, P7 SPRING_FINGERS_2

Commit message: update
Parts:
- added C1: 100nF, Capacitors_SMD:C_0805, symbol C_Small
- added C2: 10uF, Capacitors_SMD:C_0805, symbol C_Small
- added P8: CONN_01X04, Pin_Headers:Pin_Header_Angled_1x04, symbol CONN_01X04
- added Q1, Q2: BSS138, TO_SOT_Packages_SMD:SOT-23, symbol BSS138
- added R1, R2, R3, R4: 10k, Resistors_SMD:R_0805, symbol R_Small
- added U1: LD1117S18CTR, TO_SOT_Packages_SMD:SOT-223, symbol LD1117S18CTR
Connections:
- net XTI_CLK: now reaches P6.1 (P1)
- net XTI_DAT0: now reaches P6.2 (P2)
- net XTI_RX: now reaches P6.3 (P3)
- net DAT1: now reaches P6.4 (P4)
- net DAT2: now reaches P6.5 (P5)
- net DAT3: now reaches P6.6 (P6)
- net GND: now reaches P6.7 (P7)
- net GND: now also P7.7 (P7), C1.2, C2.2, P8.4 (P4), U1.1 (GND)
- net UART3_RX: now reaches P6.8 (P8)
- net UART3_RX: now also Q1.2 (S), R1.2
- net ETMClk: now reaches P7.1 (P1)
- net ETMDa0: now reaches P7.2 (P2)
- net EMU0: now reaches P7.3 (P3)
- net ETMDa1: now reaches P7.4 (P4)
- net ETMDa2: now reaches P7.5 (P5)
- net ETMDa3: now reaches P7.6 (P6)
- net UART3_TX: now reaches P7.8 (P8)
- net UART3_TX: now also Q2.2 (S), R2.2
- new net +1V8: C2.1, Q1.1 (G), Q2.1 (G), R1.1, R2.1, U1.2 (VO)
- new net +5V: C1.1, P8.1 (P1), R3.1, R4.1, U1.3 (VI)
- new net PC_UART_RX: P8.3 (P3), Q2.3 (D), R4.2
- new net PC_UART_TX: P8.2 (P2), Q1.3 (D), R3.2
Other:
- moved on the sheet: P1, P2, P3, P4, P5, P6, P7
